Commit message: wh

File: jetsoncar_description/urdf/gazebo.xacro (robot description, xacro)
@@ -106,20 +106,19 @@
 		<!--<turnGravityOff>false</turnGravityOff>-->
 	</gazebo>
+<!--
 	<gazebo reference="left_camera_mount">
-		<mu1 value="0.0"/> <!-- Columb friction coefficient in fdir1 direction -->
-		<mu2 value="0.0"/> <!-- Columb friction in perpendicular direction to fdir1 -->
-		<kp  value="10000000.0" /> <!-- contact stiffness -->
-		<kd  value="1.0" /> <!-- contact damping -->
+		<mu1 value="0.0"/>
+		<mu2 value="0.0"/>
+		<kp  value="10000000.0" />
+		<kd  value="1.0" />
 		<material>Gazebo/Black</material>
-		<!--<turnGravityOff>false</turnGravityOff>-->
 	</gazebo>
 	<gazebo reference="left_camera">
-		<mu1 value="0.0"/> <!-- Columb friction coefficient in fdir1 direction -->
-		<mu2 value="0.0"/> <!-- Columb friction in perpendicular direction to fdir1 -->
-		<kp  value="10000000.0" /> <!-- contact stiffness -->
-		<kd  value="1.0" /> <!-- contact damping -->
+		<mu1 value="0.0"/>
+		<mu2 value="0.0"/>
+		<kp  value="10000000.0" />
+		<kd  value="1.0" />
 		<material>Gazebo/Blue</material>
-		<!--<turnGravityOff>false</turnGravityOff>-->
-	</gazebo>
+	</gazebo> -->
 	<gazebo reference="right_camera_mount">
 		<mu1 value="0.0"/> <!-- Columb friction coefficient in fdir1 direction -->

File: jetsoncar_description/urdf/jetsoncar.xacro (robot description, xacro)
@@ -186,5 +186,5 @@
 	<xacro:wheel_transmission wheel="rear_left_wheel"/>
 	<!-- Sensors -->
-	<link name="left_camera_mount">
+	<!-- <link name="left_camera_mount">
 		<visual>
 			<material name="blue"/>
@@ -211,5 +211,5 @@
 		</inertial>
 	</link>
-	<xacro:fixed_offset_joint parent="left_camera_mount" child="left_camera" offset="0 0 ${camera_mount_height+camera_height/2}"/>
+	<xacro:fixed_offset_joint parent="left_camera_mount" child="left_camera" offset="0 0 ${camera_mount_height+camera_height/2}"/> -->
 	<link name="right_camera_mount">
 		<visual>
